File: KiCad/CAN.kicad_sch (KiCad schematic)
At the start: 2 parts, among them U1 TJA1042T

Commit message: 更新原理图
2023.4.7 23:34
Parts:
- removed U1: TJA1042T, Package_SO:SOIC-8_3.9x4.9mm_P1.27mm, symbol Interface_CAN_LIN:TJA1042T
- added C4: 0.1uF, Capacitor_SMD:C_0402_1005Metric_Pad0.74x0.62mm_HandSolder, symbol Device:C
- added C4: 4.7nF, Capacitor_SMD:C_1812_4532Metric_Pad1.57x3.40mm_HandSolder, symbol Device:C
- added R1: 60R, Resistor_SMD:R_1210_3225Metric_Pad1.30x2.65mm_HandSolder, symbol Device:R
- added U1: TJA1040T, Package_SO:SOIC-8_3.9x4.9mm_P1.27mm, symbol John1175:TJA1040
- R1: value 120R -> 60R; footprint Resistor_SMD:R_1020_2550Metric_Pad1.33x5.20mm_HandSolder -> Resistor_SMD:R_1210_3225Metric_Pad1.30x2.65mm_HandSolder
Connections:
- net CAN_RX: now also U1.4 (RXD)
- net CAN_TX: now also U1.1 (TXD)
- net at R1.1: now also U1.7 (CANH)
- net at R1.2: now also C4.1, R1.1, U1.5 (SPLIT)
- new net: R1.2, U1.6 (CANL)
- new net +5V: C4.1, U1.3 (VCC)
- new net GND: C4.2, C4.2, U1.2 (GND)
Other:
- moved on the sheet: R1

Commit message: 原理图完成
2023.4.8:8:30
Parts:
- added J4: Conn_01x02, Connector_JST:JST_NV_B02P-NV_1x02_P5.00mm_Vertical, symbol Connector_Generic:Conn_01x02
- added R4, R5: 10K, Resistor_SMD:R_0402_1005Metric_Pad0.72x0.64mm_HandSolder, symbol Device:R
- C4: footprint Capacitor_SMD:C_1812_4532Metric_Pad1.57x3.40mm_HandSolder -> Capacitor_SMD:C_1210_3225Metric_Pad1.33x2.70mm_HandSolder
- renumbered U1 to U3
Connections:
- net +5V: now also R4.1
- net GND: now also R5.2
- net at R1.1, U3.7 (CANH): now also J4.1 (Pin_1)
- net at R1.2, U3.6 (CANL): now also J4.2 (Pin_2)
- net at U3.8 (STB): now also R4.2, R5.1
Other:
- moved on the sheet: C4, R1, U3

Commit message: 更新封装
Signed-off-by: John1175 <njszhangshihan@126.com>
Parts:
- C4: symbol Device:C -> John1175:C
- J4: symbol Connector_Generic:Conn_01x02 -> John1175:Conn_01x02
- R1, R4, R5: symbol Device:R -> John1175:R
Changed lines of the file:
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@@
     (effects (font (size 1.27 1.27)) (justify right))
   )
-  (symbol (lib_id "Connector_Generic:Conn_01x02") (at 176.53 90.17 0) (unit 1)
+  (symbol (lib_id "John1175:Conn_01x02") (at 176.53 90.17 0) (unit 1)
     (in_bom yes) (on_board yes) (dnp no) (fields_autoplaced)
     (property "Reference" "J4" (at 179.07 90.805 0)
@@
     )
   )
-  (symbol (lib_id "Device:R") (at 144.78 86.36 0) (unit 1)
+  (symbol (lib_id "John1175:R") (at 144.78 86.36 0) (unit 1)
     (in_bom yes) (on_board yes) (dnp no)
     (property "Reference" "R1" (at 144.78 82.55 0)
@@
     )
   )
-  (symbol (lib_id "Device:R") (at 77.47 91.44 0) (unit 1)
+  (symbol (lib_id "John1175:R") (at 77.47 91.44 0) (unit 1)
     (in_bom no) (on_board yes) (dnp no)
     (property "Reference" "R4" (at 77.47 87.63 0)
@@
     )
   )
-  (symbol (lib_id "Device:R") (at 144.78 96.52 0) (unit 1)
+  (symbol (lib_id "John1175:R") (at 144.78 96.52 0) (unit 1)
     (in_bom yes) (on_board yes) (dnp no)
     (property "Reference" "R1" (at 144.78 92.71 0)
@@
     )
   )
-  (symbol (lib_id "Device:C") (at 100.33 72.39 0) (unit 1)
+  (symbol (lib_id "John1175:C") (at 100.33 72.39 0) (unit 1)
     (in_bom yes) (on_board yes) (dnp no)
     (property "Reference" "C4" (at 100.33 69.85 0)
@@
     )
   )
-  (symbol (lib_id "Device:R") (at 77.47 101.6 0) (unit 1)
+  (symbol (lib_id "John1175:R") (at 77.47 101.6 0) (unit 1)
     (in_bom yes) (on_board yes) (dnp no)
     (property "Reference" "R5" (at 77.47 97.79 0)
@@
     )
   )
-  (symbol (lib_id "Device:C") (at 135.89 99.06 0) (unit 1)
+  (symbol (lib_id "John1175:C") (at 135.89 99.06 0) (unit 1)
     (in_bom yes) (on_board yes) (dnp no)
     (property "Reference" "C4" (at 135.89 96.52 0)

Commit message: PCB更新
Parts:
- C4: symbol John1175:C -> Library:C
- J5: renamed from J4; symbol John1175:Conn_01x02 -> Library:Conn_01x02
- R1, R4, R5: symbol John1175:R -> Library:R
- U3: symbol John1175:TJA1040 -> Library:TJA1040
Changed lines of the file:
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@@
     (effects (font (size 1.27 1.27)) (justify right))
   )
-  (symbol (lib_id "John1175:Conn_01x02") (at 176.53 90.17 0) (unit 1)
-    (in_bom yes) (on_board yes) (dnp no) (fields_autoplaced)
-    (property "Reference" "J4" (at 179.07 90.805 0)
+  (symbol (lib_id "Library:Conn_01x02") (at 176.53 90.17 0) (unit 1)
+    (in_bom yes) (on_board yes) (dnp no) (fields_autoplaced)
+    (property "Reference" "J5" (at 179.07 90.805 0)
       (effects (font (size 1.27 1.27)) (justify left))
     )
@@
       (project "MM32F0140_CAN_Core"
         (path "/325db86e-5883-4f53-9728-9eee822c47e5/12a3c03d-cab3-4bb3-bab8-c4b890760701"
-          (reference "J4") (unit 1)
+          (reference "J5") (unit 1)
         )
       )
@@
         )
         (path "/325db86e-5883-4f53-9728-9eee822c47e5/12a3c03d-cab3-4bb3-bab8-c4b890760701"
-          (reference "#PWR034") (unit 1)
+          (reference "#PWR037") (unit 1)
         )
       )
@@
         )
         (path "/325db86e-5883-4f53-9728-9eee822c47e5/12a3c03d-cab3-4bb3-bab8-c4b890760701"
-          (reference "#PWR035") (unit 1)
-        )
-      )
-    )
-  )
-  (symbol (lib_id "John1175:R") (at 144.78 86.36 0) (unit 1)
+          (reference "#PWR038") (unit 1)
+        )
+      )
+    )
+  )
+  (symbol (lib_id "Library:R") (at 144.78 86.36 0) (unit 1)
     (in_bom yes) (on_board yes) (dnp no)
     (property "Reference" "R1" (at 144.78 82.55 0)
@@
         )
         (path "/325db86e-5883-4f53-9728-9eee822c47e5/12a3c03d-cab3-4bb3-bab8-c4b890760701"
-          (reference "R9") (unit 1)
-        )
-      )
-    )
-  )
-  (symbol (lib_id "John1175:R") (at 77.47 91.44 0) (unit 1)
+          (reference "R14") (unit 1)
+        )
+      )
+    )
+  )
+  (symbol (lib_id "Library:R") (at 77.47 91.44 0) (unit 1)
     (in_bom no) (on_board yes) (dnp no)
     (property "Reference" "R4" (at 77.47 87.63 0)
@@
         )
         (path "/325db86e-5883-4f53-9728-9eee822c47e5/12a3c03d-cab3-4bb3-bab8-c4b890760701"
-          (reference "R10") (unit 1)
-        )
-      )
-    )
-  )
-  (symbol (lib_id "John1175:R") (at 144.78 96.52 0) (unit 1)
+          (reference "R15") (unit 1)
+        )
+      )
+    )
+  )
+  (symbol (lib_id "Library:R") (at 144.78 96.52 0) (unit 1)
     (in_bom yes) (on_board yes) (dnp no)
     (property "Reference" "R1" (at 144.78 92.71 0)
@@
         )
         (path "/325db86e-5883-4f53-9728-9eee822c47e5/12a3c03d-cab3-4bb3-bab8-c4b890760701"
-          (reference "R11") (unit 1)
-        )
-      )
-    )
-  )
-  (symbol (lib_id "John1175:C") (at 100.33 72.39 0) (unit 1)
+          (reference "R16") (unit 1)
+        )
+      )
+    )
+  )
+  (symbol (lib_id "Library:C") (at 100.33 72.39 0) (unit 1)
     (in_bom yes) (on_board yes) (dnp no)
     (property "Reference" "C4" (at 100.33 69.85 0)
@@
         )
         (path "/325db86e-5883-4f53-9728-9eee822c47e5/12a3c03d-cab3-4bb3-bab8-c4b890760701"
-          (reference "#PWR030") (unit 1)
-        )
-      )
-    )
-  )
-  (symbol (lib_id "John1175:TJA1040") (at 116.84 91.44 0) (unit 1)
+          (reference "#PWR033") (unit 1)
+        )
+      )
+    )
+  )
+  (symbol (lib_id "Library:TJA1040") (at 116.84 91.44 0) (unit 1)
     (in_bom yes) (on_board yes) (dnp no) (fields_autoplaced)
     (property "Reference" "U3" (at 118.7959 80.01 0)
@@
         )
         (path "/325db86e-5883-4f53-9728-9eee822c47e5/12a3c03d-cab3-4bb3-bab8-c4b890760701"
-          (reference "#PWR032") (unit 1)
+          (reference "#PWR035") (unit 1)
         )
       )
@@
         )
         (path "/325db86e-5883-4f53-9728-9eee822c47e5/12a3c03d-cab3-4bb3-bab8-c4b890760701"
-          (reference "#PWR031") (unit 1)
-        )
-      )
-    )
-  )
-  (symbol (lib_id "John1175:R") (at 77.47 101.6 0) (unit 1)
+          (reference "#PWR034") (unit 1)
+        )
+      )
+    )
+  )
+  (symbol (lib_id "Library:R") (at 77.47 101.6 0) (unit 1)
     (in_bom yes) (on_board yes) (dnp no)
     (property "Reference" "R5" (at 77.47 97.79 0)
@@
         )
         (path "/325db86e-5883-4f53-9728-9eee822c47e5/12a3c03d-cab3-4bb3-bab8-c4b890760701"
-          (reference "R12") (unit 1)
+          (reference "R17") (unit 1)
         )
       )
@@
         )
         (path "/325db86e-5883-4f53-9728-9eee822c47e5/12a3c03d-cab3-4bb3-bab8-c4b890760701"
-          (reference "#PWR033") (unit 1)
-        )
-      )
-    )
-  )
-  (symbol (lib_id "John1175:C") (at 135.89 99.06 0) (unit 1)
+          (reference "#PWR036") (unit 1)
+        )
+      )
+    )
+  )
+  (symbol (lib_id "Library:C") (at 135.89 99.06 0) (unit 1)
     (in_bom yes) (on_board yes) (dnp no)
     (property "Reference" "C4" (at 135.89 96.52 0)
