File: KiCad/USB.kicad_sch (KiCad schematic)
At the start: 4 parts, among them J1 USB_C_Receptacle_USB2.0, U2 AMS1117

Commit message: 更新原理图
2023.4.7 23:34
Parts:
- added C1 (x4): 0.1uF, Capacitor_SMD:C_0402_1005Metric_Pad0.74x0.62mm_HandSolder, symbol Device:C
- added C1: 0.47uF, Capacitor_SMD:C_0402_1005Metric_Pad0.74x0.62mm_HandSolder, symbol Device:C
- added C7 (x3): 10uF, Capacitor_SMD:C_0603_1608Metric_Pad1.08x0.95mm_HandSolder, symbol Device:C
- added R1: 0R, Resistor_SMD:R_0805_2012Metric_Pad1.20x1.40mm_HandSolder, symbol Device:R
- added U3: CH340C, Package_SO:SOIC-16_3.9x9.9mm_P1.27mm, symbol Interface_USB:CH340C
- U2: now left out of the parts list
Connections:
- net +5V: now also U2.3 (VI), C1.1, C1.1, C7.1, U3.16 (VCC)
- net VCC: now also U2.2 (VO), C1.1, C7.1
- net GND: now reaches U2.1 (ADJ)
- net GND: now also J1.A1 (GND), J1.A12 (GND), J1.B1 (GND), J1.B12 (GND), C1.2, C1.2, C1.2, C1.2, C7.2, C7.2, R1.1, U3.1 (GND), U3.10 (~{DSR})
- net D+: now reaches J1.A6 (D+)
- net D+: now also J1.B6 (D+), U3.6 (UD-)
- net D-: now reaches J1.A7 (D-)
- net D-: now also J1.B7 (D-), U3.5 (UD+)
- new net: C1.1, U3.4 (V3)
- new net UART3_RX: U3.3 (RXD)
- new net UART3_TX: U3.2 (TXD)
- new net VSS: R1.2
- no-connect marks 0 -> 6
Other:
- moved on the sheet: J1, R1, U2

Commit message: 原理图完成
2023.4.8:8:30
Parts:
- added R1 (x2): 5.1K, Resistor_SMD:R_0402_1005Metric_Pad0.72x0.64mm_HandSolder, symbol Device:R
- renumbered J1 to J3, U3 to U1
Connections:
- net +5V: now also C1.1, C7.1, J3.A4 (VBUS), J3.A9 (VBUS), J3.B4 (VBUS), J3.B9 (VBUS)
- net GND: now also C1.2, C7.2, J3.S1 (SHIELD), R1.2, R1.2; no longer U1.10 (~{DSR})
- net at J3.A5 (CC1): now also R1.1
- net at J3.B5 (CC2): now also R1.1
- no-connect marks 6 -> 9
Other:
- moved on the sheet: R1

Commit message: 更新封装
Signed-off-by: John1175 <njszhangshihan@126.com>
Parts:
- removed J3: USB_C_Receptacle_USB2.0, symbol Connector:USB_C_Receptacle_USB2.0
- added J3: USB_C_Receptacle_USB2.0, John1175:USB_C_Receptacle_HRO_TYPE-C-31-M-12, symbol John1175:USB_C_Receptacle_USB2.0
- C1, C7: symbol Device:C -> John1175:C
- R1: symbol Device:R -> John1175:R
- U1: symbol Interface_USB:CH340C -> John1175:CH340C
- U2: symbol Regulator_Linear:AMS1117 -> John1175:AMS1117
Connections:
- net +5V: now also J3.A4 (VBUS), J3.A9 (VBUS), J3.B4 (VBUS), J3.B9 (VBUS)
- net D+: now also J3.A6 (D+), J3.B6 (D+)
- net D-: now also J3.A7 (D-), J3.B7 (D-)
- net GND: now also J3.A1 (GND), J3.A12 (GND), J3.B1 (GND), J3.B12 (GND), J3.S1 (SHIELD)
- net at R1.1: now also J3.A5 (CC1)
- net at R1.1: now also J3.B5 (CC2)

Commit message: 昨日修改
Parts:
- added D1: LED, symbol John1175:LED
- added R1: 10K, Resistor_SMD:R_0402_1005Metric_Pad0.72x0.64mm_HandSolder, symbol John1175:R
Connections:
- net +5V: now also R1.1
- net GND: now also D1.1 (K)
- new net: D1.2 (A), R1.2
Other:
- moved on the sheet: C1, C7
Changed lines of the file:
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@@
   (junction (at 86.36 45.72) (diameter 0) (color 0 0 0 0)
   )
-  (junction (at 86.36 55.88) (diameter 0) (color 0 0 0 0)
+  (junction (at 86.36 57.15) (diameter 0) (color 0 0 0 0)
+  )
+  (junction (at 93.98 68.58) (diameter 0) (color 0 0 0 0)
   )
   (junction (at 58.42 63.5) (diameter 0) (color 0 0 0 0)
@@
   )
   (junction (at 44.45 148.59) (diameter 0) (color 0 0 0 0)
+  )
+  (junction (at 93.98 45.72) (diameter 0) (color 0 0 0 0)
   )
   (junction (at 59.69 45.72) (diameter 0) (color 0 0 0 0)
@@
     (stroke (width 0) (type default))
   )
-  (wire (pts (xy 78.74 55.88) (xy 86.36 55.88))
+  (wire (pts (xy 78.74 57.15) (xy 86.36 57.15))
     (stroke (width 0) (type default))
   )
@@
     (stroke (width 0) (type default))
   )
+  (wire (pts (xy 93.98 55.88) (xy 93.98 58.42))
+    (stroke (width 0) (type default))
+  )
+  (wire (pts (xy 86.36 45.72) (xy 93.98 45.72))
+    (stroke (width 0) (type default))
+  )
   (wire (pts (xy 24.13 20.32) (xy 27.94 20.32))
     (stroke (width 0) (type default))
@@
     (stroke (width 0) (type default))
   )
+  (wire (pts (xy 93.98 48.26) (xy 93.98 45.72))
+    (stroke (width 0) (type default))
+  )
   (wire (pts (xy 185.42 44.45) (xy 215.9 44.45))
     (stroke (width 0) (type default))
@@
     (stroke (width 0) (type default))
   )
+  (wire (pts (xy 86.36 68.58) (xy 93.98 68.58))
+    (stroke (width 0) (type default))
+  )
   (wire (pts (xy 77.47 148.59) (xy 73.66 148.59))
     (stroke (width 0) (type default))
@@
     (stroke (width 0) (type default))
   )
-  (wire (pts (xy 78.74 46.99) (xy 78.74 45.72))
-    (stroke (width 0) (type default))
-  )
-  (wire (pts (xy 78.74 54.61) (xy 78.74 55.88))
+  (wire (pts (xy 78.74 48.26) (xy 78.74 45.72))
+    (stroke (width 0) (type default))
+  )
+  (wire (pts (xy 78.74 55.88) (xy 78.74 57.15))
     (stroke (width 0) (type default))
   )
@@
     (stroke (width 0) (type default))
   )
-  (wire (pts (xy 88.9 43.18) (xy 88.9 45.72))
+  (wire (pts (xy 93.98 43.18) (xy 93.98 45.72))
+    (stroke (width 0) (type default))
+  )
+  (wire (pts (xy 93.98 68.58) (xy 93.98 66.04))
     (stroke (width 0) (type default))
   )
@@
     (stroke (width 0) (type default))
   )
-  (wire (pts (xy 86.36 46.99) (xy 86.36 45.72))
+  (wire (pts (xy 86.36 48.26) (xy 86.36 45.72))
     (stroke (width 0) (type default))
   )
@@
     (stroke (width 0) (type default))
   )
+  (wire (pts (xy 93.98 68.58) (xy 93.98 71.12))
+    (stroke (width 0) (type default))
+  )
   (wire (pts (xy 44.45 148.59) (xy 44.45 151.13))
     (stroke (width 0) (type default))
@@
     (stroke (width 0) (type default))
   )
-  (wire (pts (xy 86.36 54.61) (xy 86.36 55.88))
+  (wire (pts (xy 86.36 55.88) (xy 86.36 57.15))
     (stroke (width 0) (type default))
   )
@@
     (stroke (width 0) (type default))
   )
-  (wire (pts (xy 86.36 55.88) (xy 86.36 57.15))
-    (stroke (width 0) (type default))
-  )
-  (wire (pts (xy 88.9 45.72) (xy 86.36 45.72))
+  (wire (pts (xy 86.36 57.15) (xy 86.36 68.58))
     (stroke (width 0) (type default))
   )
@@
     )
   )
-  (symbol (lib_id "PCM_4ms_Power-symbol:GND") (at 86.36 57.15 0) (unit 1)
-    (in_bom yes) (on_board yes) (dnp no) (fields_autoplaced)
-    (property "Reference" "#PWR017" (at 86.36 63.5 0)
-      (effects (font (size 1.27 1.27)) hide)
-    )
-    (property "Value" "GND" (at 86.36 62.23 0)
-      (effects (font (size 1.27 1.27)))
-    )
-    (property "Footprint" "" (at 86.36 57.15 0)
-      (effects (font (size 1.27 1.27)) hide)
-    )
-    (property "Datasheet" "" (at 86.36 57.15 0)
+  (symbol (lib_id "PCM_4ms_Power-symbol:GND") (at 93.98 71.12 0) (unit 1)
+    (in_bom yes) (on_board yes) (dnp no) (fields_autoplaced)
+    (property "Reference" "#PWR017" (at 93.98 77.47 0)
+      (effects (font (size 1.27 1.27)) hide)
+    )
+    (property "Value" "GND" (at 93.98 76.2 0)
+      (effects (font (size 1.27 1.27)))
+    )
+    (property "Footprint" "" (at 93.98 71.12 0)
+      (effects (font (size 1.27 1.27)) hide)
+    )
+    (property "Datasheet" "" (at 93.98 71.12 0)
       (effects (font (size 1.27 1.27)) hide)
     )
@@
     )
   )
-  (symbol (lib_id "John1175:C") (at 78.74 50.8 0) (unit 1)
+  (symbol (lib_id "John1175:C") (at 78.74 52.07 0) (unit 1)
     (in_bom yes) (on_board yes) (dnp no)
-    (property "Reference" "C7" (at 78.74 48.26 0)
-      (effects (font (size 1.27 1.27)) (justify left))
-    )
-    (property "Value" "10uF" (at 78.74 53.34 0)
-      (effects (font (size 1.27 1.27)) (justify left))
-    )
-    (property "Footprint" "Capacitor_SMD:C_0603_1608Metric_Pad1.08x0.95mm_HandSolder" (at 79.7052 54.61 0)
-      (effects (font (size 1.27 1.27)) hide)
-    )
-    (property "Datasheet" "~" (at 78.74 50.8 0)
+    (property "Reference" "C7" (at 78.74 49.53 0)
+      (effects (font (size 1.27 1.27)) (justify left))
+    )
+    (property "Value" "10uF" (at 78.74 54.61 0)
+      (effects (font (size 1.27 1.27)) (justify left))
+    )
+    (property "Footprint" "Capacitor_SMD:C_0603_1608Metric_Pad1.08x0.95mm_HandSolder" (at 79.7052 55.88 0)
+      (effects (font (size 1.27 1.27)) hide)
+    )
+    (property "Datasheet" "~" (at 78.74 52.07 0)
       (effects (font (size 1.27 1.27)) hide)
     )
@@
     )
   )
-  (symbol (lib_id "John1175:C") (at 86.36 50.8 0) (unit 1)
+  (symbol (lib_id "John1175:C") (at 86.36 52.07 0) (unit 1)
     (in_bom yes) (on_board yes) (dnp no)
-    (property "Reference" "C1" (at 86.36 48.26 0)
-      (effects (font (size 1.27 1.27)) (justify left))
-    )
-    (property "Value" "0.1uF" (at 86.36 53.34 0)
-      (effects (font (size 1.27 1.27)) (justify left))
-    )
-    (property "Footprint" "Capacitor_SMD:C_0402_1005Metric_Pad0.74x0.62mm_HandSolder" (at 87.3252 54.61 0)
-      (effects (font (size 1.27 1.27)) hide)
-    )
-    (property "Datasheet" "~" (at 86.36 50.8 0)
+    (property "Reference" "C1" (at 86.36 49.53 0)
+      (effects (font (size 1.27 1.27)) (justify left))
+    )
+    (property "Value" "0.1uF" (at 86.36 54.61 0)
+      (effects (font (size 1.27 1.27)) (justify left))
+    )
+    (property "Footprint" "Capacitor_SMD:C_0402_1005Metric_Pad0.74x0.62mm_HandSolder" (at 87.3252 55.88 0)
+      (effects (font (size 1.27 1.27)) hide)
+    )
+    (property "Datasheet" "~" (at 86.36 52.07 0)
       (effects (font (size 1.27 1.27)) hide)
     )
@@
     )
   )
+  (symbol (lib_id "John1175:LED") (at 93.98 62.23 90) (unit 1)
+    (in_bom yes) (on_board yes) (dnp no) (fields_autoplaced)
+    (property "Reference" "D1" (at 97.79 63.1825 90)
+      (effects (font (size 1.27 1.27)) (justify right))
+    )
+    (property "Value" "LED" (at 97.79 65.7225 90)
+      (effects (font (size 1.27 1.27)) (justify right))
+    )
+    (property "Footprint" "" (at 93.98 62.23 0)
+      (effects (font (size 1.27 1.27)) hide)
+    )
+    (property "Datasheet" "~" (at 93.98 62.23 0)
+      (effects (font (size 1.27 1.27)) hide)
+    )
+    (pin "1")
+    (pin "2")
+    (instances
+      (project "MM32F0140_CAN_Core"
+        (path "/325db86e-5883-4f53-9728-9eee822c47e5/54f85c82-d980-44eb-a404-039b58a4cb77"
+          (reference "D1") (unit 1)
+        )
+      )
+    )
+  )
   (symbol (lib_id "power:+5V") (at 34.29 146.05 0) (unit 1)
     (in_bom yes) (on_board yes) (dnp no) (fields_autoplaced)
@@
         (path "/325db86e-5883-4f53-9728-9eee822c47e5/54f85c82-d980-44eb-a404-039b58a4cb77"
           (reference "#PWR025") (unit 1)
+        )
+      )
+    )
+  )
+  (symbol (lib_id "John1175:R") (at 93.98 52.07 0) (unit 1)
+    (in_bom yes) (on_board yes) (dnp no)
+    (property "Reference" "R1" (at 93.98 48.26 0)
+      (effects (font (size 1.27 1.27)) (justify left))
+    )
+    (property "Value" "10K" (at 93.98 55.88 0)
+      (effects (font (size 1.27 1.27)) (justify left))
+    )
+    (property "Footprint" "Resistor_SMD:R_0402_1005Metric_Pad0.72x0.64mm_HandSolder" (at 92.202 52.07 90)
+      (effects (font (size 1.27 1.27)) hide)
+    )
+    (property "Datasheet" "~" (at 93.98 52.07 0)
+      (effects (font (size 1.27 1.27)) hide)
+    )
+    (pin "1")
+    (pin "2")
+    (instances
+      (project "MM32F0140_CAN_Core"
+        (path "/325db86e-5883-4f53-9728-9eee822c47e5/db129a86-7470-478a-aca7-0df8b6c7306b"
+          (reference "R1") (unit 1)
+        )
+        (path "/325db86e-5883-4f53-9728-9eee822c47e5/54f85c82-d980-44eb-a404-039b58a4cb77"
+          (reference "R13") (unit 1)
         )
       )
@@
     )
   )
-  (symbol (lib_id "power:+5V") (at 88.9 43.18 0) (unit 1)
-    (in_bom yes) (on_board yes) (dnp no) (fields_autoplaced)
-    (property "Reference" "#PWR02" (at 88.9 46.99 0)
-      (effects (font (size 1.27 1.27)) hide)
-    )
-    (property "Value" "+5V" (at 88.9 39.37 0)
-      (effects (font (size 1.27 1.27)))
-    )
-    (property "Footprint" "" (at 88.9 43.18 0)
-      (effects (font (size 1.27 1.27)) hide)
-    )
-    (property "Datasheet" "" (at 88.9 43.18 0)
-      (effects (font (size 1.27 1.27)) hide)
-    )
+  (symbol (lib_id "power:+5V") (at 93.98 43.18 0) (unit 1)
+    (in_bom yes) (on_board yes) (dnp no) (fields_autoplaced)
+    (property "Reference" "#PWR02" (at 93.98 46.99 0)
+      (effects (font (size 1.27 1.27)) hide)
+    )
+    (property "Value" "+5V" (at 93.98 39.37 0)
+      (effects (font (size 1.27 1.27)))
+    )
+    (property "Footprint" "" (at 93.98 43.18 0)
+      (effects (font (size 1.27 1.27)) hide)
+    )
+    (property "Datasheet" "" (at 93.98 43.18 0)
+      (effects (font (size 1.27 1.27)) hide)
+    )

Commit message: 更新原理图，添加BOM
Parts:
- D1: footprint (none) -> LED_SMD:LED_0805_2012Metric_Pad1.15x1.40mm_HandSolder
Changed lines of the file:
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@@
       (effects (font (size 1.27 1.27)) (justify right))
     )
-    (property "Footprint" "" (at 93.98 62.23 0)
+    (property "Footprint" "LED_SMD:LED_0805_2012Metric_Pad1.15x1.40mm_HandSolder" (at 93.98 62.23 0)
       (effects (font (size 1.27 1.27)) hide)
     )

Commit message: PCB更新
Parts:
- C1, C7: symbol John1175:C -> Library:C
- D5: renamed from D1; symbol John1175:LED -> Library:LED
- J4: renamed from J3; symbol John1175:USB_C_Receptacle_USB2.0 -> Library:USB_C_Receptacle_USB2.0
- R1: symbol John1175:R -> Library:R
- U1: symbol John1175:CH340C -> Library:CH340C
- U2: symbol John1175:AMS1117 -> Library:AMS1117
