File: KiCad/Core.kicad_sch (KiCad schematic)
At the start: 12 parts, among them IC1 MM32F0144C4P, Y1 8MHz

Commit message: 更新原理图
2023.4.7 23:34
Parts:
- added J2: Conn_02x10_Top_Bottom, symbol Connector_Generic:Conn_02x10_Top_Bottom
- added SW1: SW_Push, symbol Switch:SW_Push
Connections:
- net PA4: now reaches IC1.10 (PA4)
- net PA4: now also J2.5 (Pin_5)
- net PA5: now reaches IC1.11 (PA5)
- net PA5: now also J2.6 (Pin_6)
- net PA6: now reaches IC1.12 (PA6)
- net PA6: now also J2.7 (Pin_7)
- net PA7: now reaches IC1.13 (PA7)
- net PA7: now also J2.8 (Pin_8)
- net PB0: now reaches IC1.14 (PB0)
- net PB0: now also J2.13 (Pin_13)
- net PB1: now reaches IC1.15 (PB1)
- net PB1: now also J2.14 (Pin_14)
- net PA8: now reaches IC1.18 (PA8)
- net PA8: now also J2.9 (Pin_9)
- net PA15: now reaches IC1.25 (PA15)
- net PA15: now also J2.10 (Pin_10)
- net PB3: now reaches IC1.26 (PB3)
- net PB3: now also J2.15 (Pin_15)
- net PB4: now reaches IC1.27 (PB4)
- net PB4: now also J2.16 (Pin_16)
- net PB5: now reaches IC1.28 (PB5)
- net PB5: now also J2.17 (Pin_17)
- net PB6: now reaches IC1.29 (PB6)
- net PB6: now also J2.18 (Pin_18)
- net PB7: now reaches IC1.30 (PB7)
- net PB7: now also J2.19 (Pin_19)
- net PA0: now reaches IC1.6 (PA0-WKUP)
- net PA0: now also J2.1 (Pin_1)
- net PA1: now reaches IC1.7 (PA1)
- net PA1: now also J2.2 (Pin_2)
- net PA2: now reaches IC1.8 (PA2)
- net PA2: now also J2.3 (Pin_3)
- net PA3: now reaches IC1.9 (PA3)
- net PA3: now also J2.4 (Pin_4)
- new net +5V: J2.11 (Pin_11)
- new net GND: J2.20 (Pin_20)
- new net VCC: J2.12 (Pin_12)

Commit message: 原理图完成
2023.4.8:8:30
Parts:
- removed SW1: SW_Push, symbol Switch:SW_Push
- added J1: Conn_01x04, Connector_PinHeader_2.54mm:PinHeader_1x04_P2.54mm_Vertical, symbol Connector_Generic:Conn_01x04
- added SW1: SW_MEC_5E, Button_Switch_THT:SW_PUSH_6mm_H5mm, symbol Switch:SW_MEC_5E
- J2: footprint (none) -> Connector_PinHeader_2.54mm:PinHeader_2x10_P2.54mm_Vertical
- R2: renamed from R4; now fitted; now left out of the parts list
- Y1: footprint (none) -> Crystal:Crystal_HC49-U_Vertical
- renumbered C7 to C1, C4 to C2, C5 to C3, C6 to C4, C1 to C5, C2 to C6, C3 to C7, R5 to R3
Connections:
- net NRST: now also SW1.1, SW1.2
- net SWCLK: now also J1.3 (Pin_3)
- net SWDIO: now also J1.2 (Pin_2)
- net VCC: now also J1.1 (Pin_1)
- net VSS: now also J1.4 (Pin_4), SW1.3 (K), SW1.4 (A)
Other:
- moved on the sheet: C5, C6, C7, R1, Y1

Commit message: 更新封装
Signed-off-by: John1175 <njszhangshihan@126.com>
Parts:
- C1, C2, C3, C4, C5, C6, C7: symbol Device:C -> John1175:C
- IC1: symbol Library:MM32F0144C4P -> John1175:MM32F0144C4P
- J1: symbol Connector_Generic:Conn_01x04 -> John1175:Conn_01x04
- J2: symbol Connector_Generic:Conn_02x10_Top_Bottom -> John1175:Conn_02x10_Top_Bottom
- R1, R2, R3: symbol Device:R -> John1175:R
- SW1: symbol Switch:SW_MEC_5E -> John1175:SW_MEC_5E
- Y1: symbol Device:Crystal -> John1175:Crystal
Changed lines of the file:
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@@
     )
   )
-  (symbol (lib_id "Device:C") (at 190.5 99.06 0) (unit 1)
+  (symbol (lib_id "John1175:C") (at 190.5 99.06 0) (unit 1)
     (in_bom yes) (on_board yes) (dnp no)
     (property "Reference" "C7" (at 190.5 96.52 0)
@@
     )
   )
-  (symbol (lib_id "Device:C") (at 139.7 58.42 0) (unit 1)
+  (symbol (lib_id "John1175:C") (at 139.7 58.42 0) (unit 1)
     (in_bom yes) (on_board yes) (dnp no)
     (property "Reference" "C1" (at 139.7 55.88 0)
@@
     )
   )
-  (symbol (lib_id "Device:R") (at 139.7 82.55 0) (unit 1)
+  (symbol (lib_id "John1175:R") (at 139.7 82.55 0) (unit 1)
     (in_bom yes) (on_board yes) (dnp no)
     (property "Reference" "R1" (at 139.7 78.74 0)
@@
     )
   )
-  (symbol (lib_id "Connector_Generic:Conn_01x04") (at 240.03 43.18 0) (unit 1)
+  (symbol (lib_id "John1175:Conn_01x04") (at 240.03 43.18 0) (unit 1)
     (in_bom yes) (on_board yes) (dnp no) (fields_autoplaced)
     (property "Reference" "J1" (at 242.57 43.815 0)
@@
     )
   )
-  (symbol (lib_id "Library:MM32F0144C4P") (at 57.15 33.02 0) (unit 1)
+  (symbol (lib_id "John1175:MM32F0144C4P") (at 57.15 33.02 0) (unit 1)
     (in_bom yes) (on_board yes) (dnp no)
     (property "Reference" "IC1" (at 58.42 31.75 0)
@@
     )
   )
-  (symbol (lib_id "Device:C") (at 177.8 99.06 0) (unit 1)
+  (symbol (lib_id "John1175:C") (at 177.8 99.06 0) (unit 1)
     (in_bom yes) (on_board yes) (dnp no)
     (property "Reference" "C6" (at 177.8 96.52 0)
@@
     )
   )
-  (symbol (lib_id "Device:R") (at 139.7 130.81 0) (unit 1)
+  (symbol (lib_id "John1175:R") (at 139.7 130.81 0) (unit 1)
     (in_bom yes) (on_board yes) (dnp no)
     (property "Reference" "R3" (at 139.7 127 0)
@@
     )
   )
-  (symbol (lib_id "Device:C") (at 152.4 58.42 0) (unit 1)
+  (symbol (lib_id "John1175:C") (at 152.4 58.42 0) (unit 1)
     (in_bom yes) (on_board yes) (dnp no)
     (property "Reference" "C3" (at 152.4 55.88 0)
@@
     )
   )
-  (symbol (lib_id "Device:R") (at 139.7 120.65 0) (unit 1)
+  (symbol (lib_id "John1175:R") (at 139.7 120.65 0) (unit 1)
     (in_bom no) (on_board yes) (dnp no)
     (property "Reference" "R2" (at 139.7 116.84 0)
@@
     )
   )
-  (symbol (lib_id "Device:C") (at 158.75 58.42 0) (unit 1)
+  (symbol (lib_id "John1175:C") (at 158.75 58.42 0) (unit 1)
     (in_bom yes) (on_board yes) (dnp no)
     (property "Reference" "C4" (at 158.75 55.88 0)
@@
     )
   )
-  (symbol (lib_id "Device:C") (at 146.05 58.42 0) (unit 1)
+  (symbol (lib_id "John1175:C") (at 146.05 58.42 0) (unit 1)
     (in_bom yes) (on_board yes) (dnp no)
     (property "Reference" "C2" (at 146.05 55.88 0)
@@
     )
   )
-  (symbol (lib_id "Device:C") (at 139.7 92.71 0) (unit 1)
+  (symbol (lib_id "John1175:C") (at 139.7 92.71 0) (unit 1)
     (in_bom yes) (on_board yes) (dnp no)
     (property "Reference" "C5" (at 139.7 90.17 0)
@@
     )
   )
-  (symbol (lib_id "Switch:SW_MEC_5E") (at 149.86 93.98 270) (unit 1)
+  (symbol (lib_id "John1175:SW_MEC_5E") (at 149.86 93.98 270) (unit 1)
     (in_bom yes) (on_board yes) (dnp no) (fields_autoplaced)
     (property "Reference" "SW1" (at 156.21 93.345 90)
@@
     )
   )
-  (symbol (lib_id "Device:Crystal") (at 184.15 92.71 0) (unit 1)
+  (symbol (lib_id "John1175:Crystal") (at 184.15 92.71 0) (unit 1)
     (in_bom yes) (on_board yes) (dnp no) (fields_autoplaced)
     (property "Reference" "Y1" (at 184.15 86.36 0)
@@
     )
   )
-  (symbol (lib_id "Connector_Generic:Conn_02x10_Top_Bottom") (at 240.03 88.9 0) (unit 1)
+  (symbol (lib_id "John1175:Conn_02x10_Top_Bottom") (at 240.03 88.9 0) (unit 1)
     (in_bom yes) (on_board yes) (dnp no) (fields_autoplaced)
     (property "Reference" "J2" (at 241.3 73.66 0)

Commit message: 昨日修改
Parts:
- added D1 (x4): LED, symbol John1175:LED
- added J5: Conn_01x04, Connector_PinHeader_2.54mm:PinHeader_1x04_P2.54mm_Vertical, symbol John1175:Conn_01x04
- added R14, R15, R16, R17: 10K, Resistor_SMD:R_0402_1005Metric_Pad0.72x0.64mm_HandSolder, symbol John1175:R
- added SW2: SW_MEC_5E, Button_Switch_THT:SW_PUSH_6mm_H5mm, symbol John1175:SW_MEC_5E
Connections:
- net +5V: now also R14.1, R15.1, R16.1, R17.1
- net GND: now also SW2.3 (K), SW2.4 (A)
- new net: D1.1 (K), J5.3 (Pin_3)
- new net: D1.2 (A), R14.2
- new net: D1.1 (K), J5.4 (Pin_4), SW2.1, SW2.2
- new net: D1.2 (A), R17.2
- new net: D1.2 (A), R15.2
- new net: D1.1 (K), J5.1 (Pin_1)
- new net: D1.1 (K), J5.2 (Pin_2)
- new net: D1.2 (A), R16.2

Commit message: 更新原理图，添加BOM
Parts:
- D1: footprint (none) -> LED_SMD:LED_0805_2012Metric_Pad1.15x1.40mm_HandSolder
Changed lines of the file:
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@@
       (effects (font (size 1.27 1.27)) (justify right))
     )
-    (property "Footprint" "" (at 41.91 125.73 0)
+    (property "Footprint" "LED_SMD:LED_0805_2012Metric_Pad1.15x1.40mm_HandSolder" (at 41.91 125.73 0)
       (effects (font (size 1.27 1.27)) hide)
     )
@@
       (effects (font (size 1.27 1.27)) (justify right))
     )
-    (property "Footprint" "" (at 41.91 160.02 0)
+    (property "Footprint" "LED_SMD:LED_0805_2012Metric_Pad1.15x1.40mm_HandSolder" (at 41.91 160.02 0)
       (effects (font (size 1.27 1.27)) hide)
     )
@@
       (effects (font (size 1.27 1.27)) (justify right))
     )
-    (property "Footprint" "" (at 52.07 125.73 0)
+    (property "Footprint" "LED_SMD:LED_0805_2012Metric_Pad1.15x1.40mm_HandSolder" (at 52.07 125.73 0)
       (effects (font (size 1.27 1.27)) hide)
     )
@@
       (effects (font (size 1.27 1.27)) (justify right))
     )
-    (property "Footprint" "" (at 60.96 125.73 0)
-      (effects (font (size 1.27 1.27)) hide)
-    )
+    (property "Footprint" "LED_SMD:LED_0805_2012Metric_Pad1.15x1.40mm_HandSolder" (at 60.96 125.73 0)
+      (effects (font (size 1.27 1.27)) hide)
+    )

Commit message: PCB更新
Parts:
- removed SW1, SW2: SW_MEC_5E, Button_Switch_THT:SW_PUSH_6mm_H5mm, symbol John1175:SW_MEC_5E
- added SW1, SW2: SW_Push, Button_Switch_THT:SW_PUSH_6mm_H5mm, symbol Library:SW_Push
- C1, C2, C3, C4, C5, C6, C7: symbol John1175:C -> Library:C
- D1: symbol John1175:LED -> Library:LED
- IC1: symbol John1175:MM32F0144C4P -> Library:MM32F0144C4P
- J1: symbol John1175:Conn_01x04 -> Library:Conn_01x04
- J2: symbol John1175:Conn_02x10_Top_Bottom -> Library:Conn_02x10_Top_Bottom
- J3: renamed from J5; symbol John1175:Conn_01x04 -> Library:Conn_01x04
- R1: symbol John1175:R -> Library:R
- R2: renamed from R14; symbol John1175:R -> Library:R
- R3: renamed from R15; symbol John1175:R -> Library:R
- R4: renamed from R16; symbol John1175:R -> Library:R
- R5: renamed from R2; symbol John1175:R -> Library:R
- R6: renamed from R3; symbol John1175:R -> Library:R
- R7: renamed from R17; symbol John1175:R -> Library:R
- Y1: symbol John1175:Crystal -> Library:Crystal
Connections:
- net GND: now also SW2.2
- net NRST: now also SW1.1
- net VSS: now also SW1.2
- net at D1.1 (K), J3.4 (Pin_4): now also SW2.1

Commit message: PCB基本完成
Connections:
- net +5V: now also J1.1 (Pin_1)
- net GND: now also J1.4 (Pin_4)
- net VCC: no longer J1.1 (Pin_1)
- net VSS: no longer J1.4 (Pin_4)
Changed lines of the file:
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@@
     )
   )
-  (symbol (lib_id "power:VSS") (at 232.41 50.8 180) (unit 1)
-    (in_bom yes) (on_board yes) (dnp no) (fields_autoplaced)
-    (property "Reference" "#PWR03" (at 232.41 46.99 0)
-      (effects (font (size 1.27 1.27)) hide)
-    )
-    (property "Value" "VSS" (at 232.41 55.88 0)
+  (symbol (lib_id "power:+5V") (at 254 76.2 0) (unit 1)
+    (in_bom yes) (on_board yes) (dnp no) (fields_autoplaced)
+    (property "Reference" "#PWR06" (at 254 80.01 0)
+      (effects (font (size 1.27 1.27)) hide)
+    )
+    (property "Value" "+5V" (at 254 72.39 0)
+      (effects (font (size 1.27 1.27)))
+    )
+    (property "Footprint" "" (at 254 76.2 0)
+      (effects (font (size 1.27 1.27)) hide)
+    )
+    (property "Datasheet" "" (at 254 76.2 0)
+      (effects (font (size 1.27 1.27)) hide)
+    )
+    (pin "1")
+    (instances
+      (project "MM32F0140_CAN_Core"
+        (path "/325db86e-5883-4f53-9728-9eee822c47e5/db129a86-7470-478a-aca7-0df8b6c7306b"
+          (reference "#PWR06") (unit 1)
+        )
+        (path "/325db86e-5883-4f53-9728-9eee822c47e5/54f85c82-d980-44eb-a404-039b58a4cb77"
+          (reference "#PWR07") (unit 1)
+        )
+      )
+    )
+  )
+  (symbol (lib_id "power:VSS") (at 158.75 64.77 180) (unit 1)
+    (in_bom yes) (on_board yes) (dnp no) (fields_autoplaced)
+    (property "Reference" "#PWR05" (at 158.75 60.96 0)
+      (effects (font (size 1.27 1.27)) hide)
+    )
+    (property "Value" "VSS" (at 158.75 69.85 0)
+      (effects (font (size 1.27 1.27)))
+    )
+    (property "Footprint" "" (at 158.75 64.77 0)
+      (effects (font (size 1.27 1.27)) hide)
+    )
+    (property "Datasheet" "" (at 158.75 64.77 0)
+      (effects (font (size 1.27 1.27)) hide)
+    )
+    (pin "1")
+    (instances
+      (project "MM32F0140_CAN_Core"
+        (path "/325db86e-5883-4f53-9728-9eee822c47e5/db129a86-7470-478a-aca7-0df8b6c7306b"
+          (reference "#PWR05") (unit 1)
+        )
+      )
+    )
+  )
+  (symbol (lib_id "power:VDD") (at 66.04 25.4 0) (unit 1)
+    (in_bom yes) (on_board yes) (dnp no) (fields_autoplaced)
+    (property "Reference" "#PWR01" (at 66.04 29.21 0)
+      (effects (font (size 1.27 1.27)) hide)
+    )
+    (property "Value" "VDD" (at 66.04 21.59 0)
+      (effects (font (size 1.27 1.27)))
+    )
+    (property "Footprint" "" (at 66.04 25.4 0)
+      (effects (font (size 1.27 1.27)) hide)
+    )
+    (property "Datasheet" "" (at 66.04 25.4 0)
+      (effects (font (size 1.27 1.27)) hide)
+    )
+    (pin "1")
+    (instances
+      (project "MM32F0140_CAN_Core"
+        (path "/325db86e-5883-4f53-9728-9eee822c47e5/db129a86-7470-478a-aca7-0df8b6c7306b"
+          (reference "#PWR01") (unit 1)
+        )
+      )
+    )
+  )
+  (symbol (lib_id "PCM_4ms_Power-symbol:GND") (at 232.41 50.8 0) (unit 1)
+    (in_bom yes) (on_board yes) (dnp no) (fields_autoplaced)
+    (property "Reference" "#PWR017" (at 232.41 57.15 0)
+      (effects (font (size 1.27 1.27)) hide)
+    )
+    (property "Value" "GND" (at 232.41 55.88 0)
       (effects (font (size 1.27 1.27)))
     )
@@
     (instances
       (project "MM32F0140_CAN_Core"
+        (path "/325db86e-5883-4f53-9728-9eee822c47e5/54f85c82-d980-44eb-a404-039b58a4cb77"
+          (reference "#PWR017") (unit 1)
+        )
         (path "/325db86e-5883-4f53-9728-9eee822c47e5/db129a86-7470-478a-aca7-0df8b6c7306b"
           (reference "#PWR03") (unit 1)
@@
     )
   )
-  (symbol (lib_id "power:+5V") (at 254 76.2 0) (unit 1)
-    (in_bom yes) (on_board yes) (dnp no) (fields_autoplaced)
-    (property "Reference" "#PWR06" (at 254 80.01 0)
-      (effects (font (size 1.27 1.27)) hide)
-    )
-    (property "Value" "+5V" (at 254 72.39 0)
-      (effects (font (size 1.27 1.27)))
-    )
-    (property "Footprint" "" (at 254 76.2 0)
-      (effects (font (size 1.27 1.27)) hide)
-    )
-    (property "Datasheet" "" (at 254 76.2 0)
-      (effects (font (size 1.27 1.27)) hide)
-    )
-    (pin "1")
-    (instances
-      (project "MM32F0140_CAN_Core"
-        (path "/325db86e-5883-4f53-9728-9eee822c47e5/db129a86-7470-478a-aca7-0df8b6c7306b"
-          (reference "#PWR06") (unit 1)
-        )
-        (path "/325db86e-5883-4f53-9728-9eee822c47e5/54f85c82-d980-44eb-a404-039b58a4cb77"
-          (reference "#PWR07") (unit 1)
-        )
-      )
-    )
-  )
-  (symbol (lib_id "power:VSS") (at 158.75 64.77 180) (unit 1)
-    (in_bom yes) (on_board yes) (dnp no) (fields_autoplaced)
-    (property "Reference" "#PWR05" (at 158.75 60.96 0)
-      (effects (font (size 1.27 1.27)) hide)
-    )
-    (property "Value" "VSS" (at 158.75 69.85 0)
-      (effects (font (size 1.27 1.27)))
-    )
-    (property "Footprint" "" (at 158.75 64.77 0)
-      (effects (font (size 1.27 1.27)) hide)
-    )
-    (property "Datasheet" "" (at 158.75 64.77 0)
-      (effects (font (size 1.27 1.27)) hide)
-    )
-    (pin "1")
-    (instances
-      (project "MM32F0140_CAN_Core"
-        (path "/325db86e-5883-4f53-9728-9eee822c47e5/db129a86-7470-478a-aca7-0df8b6c7306b"
-          (reference "#PWR05") (unit 1)
-        )
-      )
-    )
-  )
-  (symbol (lib_id "power:VDD") (at 66.04 25.4 0) (unit 1)
-    (in_bom yes) (on_board yes) (dnp no) (fields_autoplaced)
-    (property "Reference" "#PWR01" (at 66.04 29.21 0)
-      (effects (font (size 1.27 1.27)) hide)
-    )
-    (property "Value" "VDD" (at 66.04 21.59 0)
-      (effects (font (size 1.27 1.27)))
-    )
-    (property "Footprint" "" (at 66.04 25.4 0)
-      (effects (font (size 1.27 1.27)) hide)
-    )
-    (property "Datasheet" "" (at 66.04 25.4 0)
-      (effects (font (size 1.27 1.27)) hide)
-    )
-    (pin "1")
-    (instances
-      (project "MM32F0140_CAN_Core"
-        (path "/325db86e-5883-4f53-9728-9eee822c47e5/db129a86-7470-478a-aca7-0df8b6c7306b"
-          (reference "#PWR01") (unit 1)
-        )
-      )
-    )
-  )
   (symbol (lib_id "power:+5V") (at 41.91 109.22 0) (unit 1)
     (in_bom yes) (on_board yes) (dnp no) (fields_autoplaced)
@@
         (path "/325db86e-5883-4f53-9728-9eee822c47e5/54f85c82-d980-44eb-a404-039b58a4cb77"
           (reference "#PWR015") (unit 1)
-        )
-      )
-    )
-  )
-  (symbol (lib_id "power:VCC") (at 232.41 38.1 0) (unit 1)
-    (in_bom yes) (on_board yes) (dnp no) (fields_autoplaced)
-    (property "Reference" "#PWR08" (at 232.41 41.91 0)
-      (effects (font (size 1.27 1.27)) hide)
-    )
-    (property "Value" "VCC" (at 232.41 34.29 0)
-      (effects (font (size 1.27 1.27)))
-    )
-    (property "Footprint" "" (at 232.41 38.1 0)
-      (effects (font (size 1.27 1.27)) hide)
-    )
-    (property "Datasheet" "" (at 232.41 38.1 0)
-      (effects (font (size 1.27 1.27)) hide)
-    )
-    (pin "1")
-    (instances
-      (project "MM32F0140_CAN_Core"
-        (path "/325db86e-5883-4f53-9728-9eee822c47e5/54f85c82-d980-44eb-a404-039b58a4cb77"
-          (reference "#PWR08") (unit 1)
-        )
-        (path "/325db86e-5883-4f53-9728-9eee822c47e5/db129a86-7470-478a-aca7-0df8b6c7306b"
-          (reference "#PWR02") (unit 1)
         )
       )
@@
         )
       )
+    )
+  )
+  (symbol (lib_id "power:+5V") (at 232.41 38.1 0) (unit 1)
+    (in_bom yes) (on_board yes) (dnp no) (fields_autoplaced)
+    (property "Reference" "#PWR02" (at 232.41 41.91 0)
+      (effects (font (size 1.27 1.27)) hide)
+    )
+    (property "Value" "+5V" (at 232.41 34.29 0)
+      (effects (font (size 1.27 1.27)))
+    )
+    (property "Footprint" "" (at 232.41 38.1 0)
+      (effects (font (size 1.27 1.27)) hide)
+    )
+    (property "Datasheet" "" (at 232.41 38.1 0)
+      (effects (font (size 1.27 1.27)) hide)
+    )
+    (pin "1")
+    (instances
+      (project "MM32F0140_CAN_Core"
+        (path "/325db86e-5883-4f53-9728-9eee822c47e5/db129a86-7470-478a-aca7-0df8b6c7306b"
+          (reference "#PWR02") (unit 1)
+        )
+        (path "/325db86e-5883-4f53-9728-9eee822c47e5/54f85c82-d980-44eb-a404-039b58a4cb77"
+          (reference "#PWR07") (unit 1)
+        )
+      )
