File: KiCad/MM32F0140_CAN_Core.kicad_pcb (KiCad board)
At the start: 2 copper layers, 1 part, among them IC1 MM32F0144C4P

Commit message: 更新原理图
2023.4.7 23:34
Parts:
- added C1: 0.1uF, Capacitor_SMD:C_0402_1005Metric_Pad0.74x0.62mm_HandSolder, F.Cu at (152.8, 77.6)
- added C10: 10uF, Capacitor_SMD:C_0603_1608Metric_Pad1.08x0.95mm_HandSolder, F.Cu at (133.1, 74.1)
- added C11: 10uF, Capacitor_SMD:C_0603_1608Metric_Pad1.08x0.95mm_HandSolder, F.Cu at (133.1, 76.6)
- added C12: 10uF, Capacitor_SMD:C_0603_1608Metric_Pad1.08x0.95mm_HandSolder, F.Cu at (133.1, 79.1)
- added C13: 0.1uF, Capacitor_SMD:C_0402_1005Metric_Pad0.74x0.62mm_HandSolder, F.Cu at (141.0, 74.6)
- added C15: 0.1uF, Capacitor_SMD:C_0402_1005Metric_Pad0.74x0.62mm_HandSolder, F.Cu at (141.0, 76.5)
- added C16: 0.47uF, Capacitor_SMD:C_0402_1005Metric_Pad0.74x0.62mm_HandSolder, F.Cu at (141.0, 78.5)
- added C2: 22pF, Capacitor_SMD:C_0402_1005Metric_Pad0.74x0.62mm_HandSolder, F.Cu at (152.8, 79.5)
- added C3: 22pF, Capacitor_SMD:C_0402_1005Metric_Pad0.74x0.62mm_HandSolder, F.Cu at (152.8, 81.5)
- added C4: 0.1uF, Capacitor_SMD:C_0402_1005Metric_Pad0.74x0.62mm_HandSolder, F.Cu at (152.8, 83.5)
- added C5: 0.1uF, Capacitor_SMD:C_0402_1005Metric_Pad0.74x0.62mm_HandSolder, F.Cu at (152.8, 85.5)
- added C6: 0.1uF, Capacitor_SMD:C_0402_1005Metric_Pad0.74x0.62mm_HandSolder, F.Cu at (152.8, 87.4)
- added C7: 10uF, Capacitor_SMD:C_0603_1608Metric_Pad1.08x0.95mm_HandSolder, F.Cu at (156.6, 83.8)
- added C8: 0.1uF, Capacitor_SMD:C_0402_1005Metric_Pad0.74x0.62mm_HandSolder, F.Cu at (141.0, 70.6)
- added C9: 0.1uF, Capacitor_SMD:C_0402_1005Metric_Pad0.74x0.62mm_HandSolder, F.Cu at (141.0, 72.6)
- added R1: 100K, Resistor_SMD:R_0402_1005Metric_Pad0.72x0.64mm_HandSolder, F.Cu at (156.1, 77.6)
- added R2: 0R, Resistor_SMD:R_0805_2012Metric_Pad1.20x1.40mm_HandSolder, F.Cu at (145.0, 71.1)
- added R3: 0R, Resistor_SMD:R_0805_2012Metric_Pad1.20x1.40mm_HandSolder, F.Cu at (145.0, 74.1)
- added R4: 10K, Resistor_SMD:R_0402_1005Metric_Pad0.72x0.64mm_HandSolder, F.Cu at (156.1, 79.6)
- added R5: 10K, Resistor_SMD:R_0402_1005Metric_Pad0.72x0.64mm_HandSolder, F.Cu at (156.1, 81.6)
- added R6: 120R, Resistor_SMD:R_1210_3225Metric_Pad1.30x2.65mm_HandSolder, F.Cu at (153.9, 71.2)
- added R7: 0R, Resistor_SMD:R_0805_2012Metric_Pad1.20x1.40mm_HandSolder, F.Cu at (145.0, 77.0)
- added U1: TJA1042T, Package_SO:SOIC-8_3.9x4.9mm_P1.27mm, F.Cu at (155.5, 64.6)
- added U2: AMS1117, Package_TO_SOT_SMD:SOT-223-3_TabPin2, F.Cu at (144.3, 65.5)
- added U3: CH340C, Package_SO:SOIC-16_3.9x9.9mm_P1.27mm, F.Cu at (135.2, 67.1)
- IC1: footprint Library:LQFP-32_7x7mm_P0.8mm -> Package_QFP:LQFP-32_7x7mm_P0.8mm
- moved IC1 4.90 mm to (119.4, 76.2)
Connections:
- IC1 pad 1: unconnected-(IC1-VDD_1-Pad1) -> VDD
- IC1 pad 10: unconnected-(IC1-PA4-Pad10) -> /Core/PA4
- IC1 pad 11: unconnected-(IC1-PA5-Pad11) -> /Core/PA5
- IC1 pad 12: unconnected-(IC1-PA6-Pad12) -> /Core/PA6
- IC1 pad 13: unconnected-(IC1-PA7-Pad13) -> /Core/PA7
- IC1 pad 14: unconnected-(IC1-PB0-Pad14) -> /Core/PB0
- IC1 pad 15: unconnected-(IC1-PB1-Pad15) -> /Core/PB1
- IC1 pad 16: unconnected-(IC1-VSS_1-Pad16) -> VSS
- IC1 pad 17: unconnected-(IC1-VDD_2-Pad17) -> VDD
- IC1 pad 18: unconnected-(IC1-PA8-Pad18) -> /Core/PA8
- IC1 pad 19: unconnected-(IC1-PA9-Pad19) -> /Core/CAN_RX
- IC1 pad 2: unconnected-(IC1-PD0-OSC_IN-Pad2) -> /Core/OSC_I
- IC1 pad 20: unconnected-(IC1-PA10-Pad20) -> /Core/CAN_TX
- IC1 pad 21: unconnected-(IC1-PA11-Pad21) -> /Core/UART3_TX
- IC1 pad 22: unconnected-(IC1-PA12-Pad22) -> /Core/UART3_RX
- IC1 pad 23: unconnected-(IC1-PA13-Pad23) -> /Core/SWDIO
- IC1 pad 24: unconnected-(IC1-PA14-Pad24) -> /Core/SWCLK
- IC1 pad 25: unconnected-(IC1-PA15-Pad25) -> /Core/PA15
- IC1 pad 26: unconnected-(IC1-PB3-Pad26) -> /Core/PB3
- IC1 pad 27: unconnected-(IC1-PB4-Pad27) -> /Core/PB4
- IC1 pad 28: unconnected-(IC1-PB5-Pad28) -> /Core/PB5
- IC1 pad 29: unconnected-(IC1-PB6-Pad29) -> /Core/PB6
- IC1 pad 3: unconnected-(IC1-PD1-OSC_OUT-Pad3) -> /Core/OSC_O
- IC1 pad 30: unconnected-(IC1-PB7-Pad30) -> /Core/PB7
- IC1 pad 31: unconnected-(IC1-PD5-BOOT0-Pad31) -> /Core/BOOT0
- IC1 pad 32: unconnected-(IC1-VSS_2-Pad32) -> VSS
- IC1 pad 4: unconnected-(IC1-NRST1-Pad4) -> /Core/NRST
- IC1 pad 5: unconnected-(IC1-VDDA-Pad5) -> VDD
- IC1 pad 6: unconnected-(IC1-PA0-WKUP-Pad6) -> /Core/PA0
- IC1 pad 7: unconnected-(IC1-PA1-Pad7) -> /Core/PA1
- IC1 pad 8: unconnected-(IC1-PA2-Pad8) -> /Core/PA2
- IC1 pad 9: unconnected-(IC1-PA3-Pad9) -> /Core/PA3

Commit message: 原理图完成
2023.4.8:8:30
Parts:
- added C16: 0.1uF, Capacitor_SMD:C_0402_1005Metric_Pad0.74x0.62mm_HandSolder, F.Cu at (111.6, 57.1)
- added C17: 4.7nF, Capacitor_SMD:C_1812_4532Metric_Pad1.57x3.40mm_HandSolder, F.Cu at (109.6, 61.0)
- added J1: Conn_01x04, Connector_PinHeader_2.54mm:PinHeader_1x04_P2.54mm_Vertical, F.Cu at (84.8, 50.3)
- added J2: Conn_02x10_Top_Bottom, Connector_PinHeader_2.54mm:PinHeader_2x10_P2.54mm_Vertical, F.Cu at (77.6, 50.3)
- added J4: Conn_01x02, Connector_JST:JST_NV_B02P-NV_1x02_P5.00mm_Vertical, F.Cu at (101.4, 52.7)
- added R10: 10K, Resistor_SMD:R_0402_1005Metric_Pad0.72x0.64mm_HandSolder, F.Cu at (111.6, 53.1)
- added R11: 60R, Resistor_SMD:R_1210_3225Metric_Pad1.30x2.65mm_HandSolder, F.Cu at (112.9, 50.0)
- added R12: 10K, Resistor_SMD:R_0402_1005Metric_Pad0.72x0.64mm_HandSolder, F.Cu at (111.6, 55.1)
- added R4: 5.1K, Resistor_SMD:R_0402_1005Metric_Pad0.72x0.64mm_HandSolder, F.Cu at (99.1, 67.9)
- added R5: 5.1K, Resistor_SMD:R_0402_1005Metric_Pad0.72x0.64mm_HandSolder, F.Cu at (99.1, 69.9)
- added SW1: SW_MEC_5E, Button_Switch_THT:SW_PUSH_6mm_H5mm, F.Cu at (84.5, 62.2)
- added U3: TJA1040T, Package_SO:SOIC-8_3.9x4.9mm_P1.27mm, F.Cu at (101.7, 61.7)
- added Y1: 8MHz, Crystal:Crystal_HC49-U_Vertical, F.Cu at (86.5, 72.1)
- R9: renamed from R6; value 120R -> 60R
- renumbered C7 to C1, C16 to C10, C15 to C11, C10 to C12, C8 to C13, C9 to C14, C11 to C15, C4 to C2, C5 to C3, C6 to C4, C1 to C5, C2 to C6, C3 to C7, C12 to C8, C13 to C9, R4 to R2, R5 to R3, R2 to R6, R3 to R7, R7 to R8, U3 to U1
Connections:
- C8 pad 1: unconnected-(C12-Pad1) -> +5V
- C8 pad 2: unconnected-(C12-Pad2) -> GND
- C9 pad 1: unconnected-(C13-Pad1) -> +5V
- C9 pad 2: unconnected-(C13-Pad2) -> GND
- IC1 pad 19: /Core/CAN_RX -> /CAN/CAN_RX
- IC1 pad 20: /Core/CAN_TX -> /CAN/CAN_TX
- R9 pad 1: unconnected-(R6-Pad1) -> Net-(J4-Pin_1)
- R9 pad 2: unconnected-(R6-Pad2) -> Net-(U3-SPLIT)
- U1 pad 10: GND -> unconnected-(U1-~{DSR}-Pad10)

Commit message: 更新封装
Signed-off-by: John1175 <njszhangshihan@126.com>
Parts:
- added J3: USB_C_Receptacle_USB2.0, John1175:USB_C_Receptacle_HRO_TYPE-C-31-M-12, F.Cu at (84.6, 87.8)
- C1, C12, C15, C8: footprint Capacitor_SMD:C_0603_1608Metric_Pad1.08x0.95mm_HandSolder -> John1175:C_0603_1608Metric_Pad1.08x0.95mm_HandSolder
- C10, C11, C13, C14, C16, C2, C3, C4, C5, C6, C7, C9: footprint Capacitor_SMD:C_0402_1005Metric_Pad0.74x0.62mm_HandSolder -> John1175:C_0402_1005Metric_Pad0.74x0.62mm_HandSolder
- C17: footprint Capacitor_SMD:C_1812_4532Metric_Pad1.57x3.40mm_HandSolder -> John1175:C_1210_3225Metric_Pad1.33x2.70mm_HandSolder
- IC1: footprint Package_QFP:LQFP-32_7x7mm_P0.8mm -> John1175:LQFP-32_7x7mm_P0.8mm
- J1: footprint Connector_PinHeader_2.54mm:PinHeader_1x04_P2.54mm_Vertical -> John1175:PinHeader_1x04_P2.54mm_Vertical
- J2: footprint Connector_PinHeader_2.54mm:PinHeader_2x10_P2.54mm_Vertical -> John1175:PinHeader_2x10_P2.54mm_Vertical
- J4: footprint Connector_JST:JST_NV_B02P-NV_1x02_P5.00mm_Vertical -> John1175:JST_NV_B02P-NV_1x02_P5.00mm_Vertical
- R1, R10, R12, R2, R3, R4, R5: footprint Resistor_SMD:R_0402_1005Metric_Pad0.72x0.64mm_HandSolder -> John1175:R_0402_1005Metric_Pad0.72x0.64mm_HandSolder
- R11, R9: footprint Resistor_SMD:R_1210_3225Metric_Pad1.30x2.65mm_HandSolder -> John1175:R_1210_3225Metric_Pad1.30x2.65mm_HandSolder
- R6, R7, R8: footprint Resistor_SMD:R_0805_2012Metric_Pad1.20x1.40mm_HandSolder -> John1175:R_0805_2012Metric_Pad1.20x1.40mm_HandSolder
- SW1: footprint Button_Switch_THT:SW_PUSH_6mm_H5mm -> John1175:SW_PUSH_6mm_H5mm
- U1: footprint Package_SO:SOIC-16_3.9x9.9mm_P1.27mm -> John1175:SOIC-16_3.9x9.9mm_P1.27mm
- U1, U3: footprint Package_SO:SOIC-8_3.9x4.9mm_P1.27mm -> John1175:SOIC-8_3.9x4.9mm_P1.27mm
- U2: footprint Package_TO_SOT_SMD:SOT-223-3_TabPin2 -> John1175:SOT-223-3_TabPin2
- Y1: footprint Crystal:Crystal_HC49-U_Vertical -> John1175:Crystal_HC49-U_Vertical

Commit message: 昨日修改
Parts:
- removed the U1 at (155.5, 64.6)
- C1, C12, C15, C8: footprint John1175:C_0603_1608Metric_Pad1.08x0.95mm_HandSolder -> Capacitor_SMD:C_0603_1608Metric_Pad1.08x0.95mm_HandSolder
- C10, C11, C13, C14, C16, C2, C3, C4, C5, C6, C7, C9: footprint John1175:C_0402_1005Metric_Pad0.74x0.62mm_HandSolder -> Capacitor_SMD:C_0402_1005Metric_Pad0.74x0.62mm_HandSolder
- C17: footprint John1175:C_1210_3225Metric_Pad1.33x2.70mm_HandSolder -> Capacitor_SMD:C_1210_3225Metric_Pad1.33x2.70mm_HandSolder
- IC1: footprint John1175:LQFP-32_7x7mm_P0.8mm -> Package_QFP:LQFP-32_7x7mm_P0.8mm
- J1: footprint John1175:PinHeader_1x04_P2.54mm_Vertical -> Connector_PinHeader_2.54mm:PinHeader_1x04_P2.54mm_Vertical
- J2: footprint John1175:PinHeader_2x10_P2.54mm_Vertical -> Connector_PinHeader_2.54mm:PinHeader_2x10_P2.54mm_Vertical
- J4: footprint John1175:JST_NV_B02P-NV_1x02_P5.00mm_Vertical -> Connector_JST:JST_NV_B02P-NV_1x02_P5.00mm_Vertical
- R1, R10, R12, R2, R3, R4, R5: footprint John1175:R_0402_1005Metric_Pad0.72x0.64mm_HandSolder -> Resistor_SMD:R_0402_1005Metric_Pad0.72x0.64mm_HandSolder
- R11, R9: footprint John1175:R_1210_3225Metric_Pad1.30x2.65mm_HandSolder -> Resistor_SMD:R_1210_3225Metric_Pad1.30x2.65mm_HandSolder
- R6, R7, R8: footprint John1175:R_0805_2012Metric_Pad1.20x1.40mm_HandSolder -> Resistor_SMD:R_0805_2012Metric_Pad1.20x1.40mm_HandSolder
- SW1: footprint John1175:SW_PUSH_6mm_H5mm -> Button_Switch_THT:SW_PUSH_6mm_H5mm
- U1: footprint John1175:SOIC-16_3.9x9.9mm_P1.27mm -> Package_SO:SOIC-16_3.9x9.9mm_P1.27mm
- U2: footprint John1175:SOT-223-3_TabPin2 -> Package_TO_SOT_SMD:SOT-223-3_TabPin2
- U3: footprint John1175:SOIC-8_3.9x4.9mm_P1.27mm -> Package_SO:SOIC-8_3.9x4.9mm_P1.27mm
- Y1: footprint John1175:Crystal_HC49-U_Vertical -> Crystal:Crystal_HC49-U_Vertical
- moved J4 131.1 mm to (205.7, 132.1), turned to -90 degrees
- moved J3 128.7 mm to (210.9, 63.1), turned to 90 degrees
- moved R11 117.2 mm to (194.0, 134.6)
- moved C17 116.6 mm to (195.6, 139.7)
- moved U3 111.0 mm to (185.4, 134.6)
- moved R5 105.0 mm to (203.2, 55.9), turned to 90 degrees
- moved R4 102.8 mm to (201.2, 55.9), turned to 90 degrees
- moved Y1 83.9 mm to (165.1, 101.6)
- moved J2 82.2 mm to (115.6, 123.2)
- moved U2 72.6 mm to (205.7, 104.1)
- moved R9 70.8 mm to (194.0, 129.5), turned to 180 degrees
- moved IC1 62.7 mm to (142.2, 134.6)
- moved U1 60.6 mm to (195.6, 63.5), turned to 180 degrees
- moved J1 52.7 mm to (114.3, 94.0)

Commit message: PCB更新
Parts:
- added D1: LED, Library:LED_0805_2012Metric_Pad1.15x1.40mm_HandSolder, F.Cu at (28.1, 83.2)
- added D2: LED, Library:LED_0805_2012Metric_Pad1.15x1.40mm_HandSolder, F.Cu at (28.1, 86.2)
- added D3: LED, Library:LED_0805_2012Metric_Pad1.15x1.40mm_HandSolder, F.Cu at (28.1, 89.2)
- added D4: LED, Library:LED_0805_2012Metric_Pad1.15x1.40mm_HandSolder, F.Cu at (28.1, 92.3)
- added D5: LED, Library:LED_0805_2012Metric_Pad1.15x1.40mm_HandSolder, F.Cu at (34.0, 20.3)
- added J3: Conn_01x04, Library:PinHeader_1x04_P2.54mm_Vertical, F.Cu at (32.8, 84.0)
- added R2: 10K, Library:R_0402_1005Metric_Pad0.72x0.64mm_HandSolder, F.Cu at (36.8, 82.6)
- added R3: 10K, Library:R_0402_1005Metric_Pad0.72x0.64mm_HandSolder, F.Cu at (36.8, 84.6)
- added R4: 10K, Library:R_0402_1005Metric_Pad0.72x0.64mm_HandSolder, F.Cu at (36.8, 86.6)
- added R7: 10K, Library:R_0402_1005Metric_Pad0.72x0.64mm_HandSolder, F.Cu at (36.8, 88.6)
- added R8: 10K, Library:R_0402_1005Metric_Pad0.72x0.64mm_HandSolder, F.Cu at (33.2, 22.8)
- added SW2: SW_Push, Library:SW_PUSH_6mm_H5mm, F.Cu at (42.5, 89.2)
- C1, C12, C15, C8: footprint Capacitor_SMD:C_0603_1608Metric_Pad1.08x0.95mm_HandSolder -> Library:C_0603_1608Metric_Pad1.08x0.95mm_HandSolder
- C10, C11, C13, C14, C16, C2, C3, C4, C5, C6, C7, C9: footprint Capacitor_SMD:C_0402_1005Metric_Pad0.74x0.62mm_HandSolder -> Library:C_0402_1005Metric_Pad0.74x0.62mm_HandSolder
- C17: footprint Capacitor_SMD:C_1210_3225Metric_Pad1.33x2.70mm_HandSolder -> Library:C_1210_3225Metric_Pad1.33x2.70mm_HandSolder
- IC1: footprint Package_QFP:LQFP-32_7x7mm_P0.8mm -> Library:LQFP-32_7x7mm_P0.8mm
- J1: footprint Connector_PinHeader_2.54mm:PinHeader_1x04_P2.54mm_Vertical -> Library:PinHeader_1x04_P2.54mm_Vertical
- J2: footprint Connector_PinHeader_2.54mm:PinHeader_2x10_P2.54mm_Vertical -> Library:PinHeader_2x10_P2.54mm_Vertical
- J4: renamed from J3; footprint John1175:USB_C_Receptacle_HRO_TYPE-C-31-M-12 -> Library:USB_C_Receptacle_HRO_TYPE-C-31-M-12
- J5: renamed from J4; footprint Connector_JST:JST_NV_B02P-NV_1x02_P5.00mm_Vertical -> Library:JST_NV_B02P-NV_1x02_P5.00mm_Vertical
- R1: footprint Resistor_SMD:R_0402_1005Metric_Pad0.72x0.64mm_HandSolder -> Library:R_0402_1005Metric_Pad0.72x0.64mm_HandSolder
- R10: renamed from R5; footprint Resistor_SMD:R_0402_1005Metric_Pad0.72x0.64mm_HandSolder -> Library:R_0402_1005Metric_Pad0.72x0.64mm_HandSolder
- R11: renamed from R6; footprint Resistor_SMD:R_0805_2012Metric_Pad1.20x1.40mm_HandSolder -> Library:R_0805_2012Metric_Pad1.20x1.40mm_HandSolder
- R12: renamed from R7; footprint Resistor_SMD:R_0805_2012Metric_Pad1.20x1.40mm_HandSolder -> Library:R_0805_2012Metric_Pad1.20x1.40mm_HandSolder
- R13: renamed from R8; footprint Resistor_SMD:R_0805_2012Metric_Pad1.20x1.40mm_HandSolder -> Library:R_0805_2012Metric_Pad1.20x1.40mm_HandSolder
- R14: renamed from R9; footprint Resistor_SMD:R_1210_3225Metric_Pad1.30x2.65mm_HandSolder -> Library:R_1210_3225Metric_Pad1.30x2.65mm_HandSolder
- R15: renamed from R10; footprint Resistor_SMD:R_0402_1005Metric_Pad0.72x0.64mm_HandSolder -> Library:R_0402_1005Metric_Pad0.72x0.64mm_HandSolder
- R16: renamed from R11; footprint Resistor_SMD:R_1210_3225Metric_Pad1.30x2.65mm_HandSolder -> Library:R_1210_3225Metric_Pad1.30x2.65mm_HandSolder
- R17: renamed from R12; footprint Resistor_SMD:R_0402_1005Metric_Pad0.72x0.64mm_HandSolder -> Library:R_0402_1005Metric_Pad0.72x0.64mm_HandSolder
- R5: renamed from R2; footprint Resistor_SMD:R_0402_1005Metric_Pad0.72x0.64mm_HandSolder -> Library:R_0402_1005Metric_Pad0.72x0.64mm_HandSolder
- R6: renamed from R3; footprint Resistor_SMD:R_0402_1005Metric_Pad0.72x0.64mm_HandSolder -> Library:R_0402_1005Metric_Pad0.72x0.64mm_HandSolder
- R9: renamed from R4; footprint Resistor_SMD:R_0402_1005Metric_Pad0.72x0.64mm_HandSolder -> Library:R_0402_1005Metric_Pad0.72x0.64mm_HandSolder
- SW1: value SW_MEC_5E -> SW_Push; footprint Button_Switch_THT:SW_PUSH_6mm_H5mm -> Library:SW_PUSH_6mm_H5mm
- U1: footprint Package_SO:SOIC-16_3.9x9.9mm_P1.27mm -> Library:SOIC-16_3.9x9.9mm_P1.27mm
- U2: footprint Package_TO_SOT_SMD:SOT-223-3_TabPin2 -> Library:SOT-223-3_TabPin2
- U3: footprint Package_SO:SOIC-8_3.9x4.9mm_P1.27mm -> Library:SOIC-8_3.9x4.9mm_P1.27mm
- Y1: footprint Crystal:Crystal_HC49-U_Vertical -> Library:Crystal_HC49-U_Vertical
- moved C8 132.1 mm to (256.5, 32.2), turned to 90 degrees
- moved C9 125.2 mm to (259.1, 33.0), turned to 90 degrees
- moved C15 124.6 mm to (256.5, 59.3), turned to 90 degrees
- moved C12 123.8 mm to (256.5, 65.2), turned to -90 degrees
- moved C14 118.9 mm to (259.1, 59.0), turned to 90 degrees
- moved C13 118.2 mm to (259.1, 65.5), turned to -90 degrees
- moved C11 118.1 mm to (252.0, 36.2)
- moved C16 114.8 mm to (200.7, 129.5)
- moved R15 113.8 mm to (200.5, 124.3)
- moved R17 113.8 mm to (200.5, 126.2)
- moved C10 109.0 mm to (244.3, 43.8)
- moved U2 74.7 mm to (266.7, 61.0)
- moved C7 70.4 mm to (213.2, 45.2), turned to 90 degrees
- moved C5 70.0 mm to (86.3, 55.9)
- moved R1 70.0 mm to (89.5, 55.9)
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Connections:
- SW1 pad 2: /Core/NRST -> VSS

Commit message: PCB初稿
Parts:
- moved U2 158.5 mm to (112.5, 97.9), turned to 90 degrees
- moved C14 155.4 mm to (110.3, 103.8), turned to 180 degrees
- moved C15 153.3 mm to (110.6, 106.3), turned to 180 degrees
- moved C13 148.0 mm to (116.1, 103.8), turned to 0 degrees
- moved R8 147.4 mm to (158.0, 101.3), turned to 90 degrees
- moved C12 146.4 mm to (115.7, 105.1), turned to 0 degrees
- moved D5 144.6 mm to (158.0, 94.8), turned to -90 degrees
- moved D3 127.3 mm to (155.4, 94.8), turned to -90 degrees
- moved D2 124.9 mm to (152.7, 94.8), turned to -90 degrees
- moved J3 124.1 mm to (156.8, 89.9), turned to -90 degrees
- moved D1 122.5 mm to (150.1, 94.8), turned to -90 degrees
- moved J4 119.7 mm to (166.2, 92.3), turned to 180 degrees
- moved R4 119.5 mm to (155.4, 101.3), turned to 90 degrees
- moved D4 119.3 mm to (147.4, 94.8), turned to -90 degrees
- moved R3 117.1 mm to (152.7, 101.3), turned to 90 degrees
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Routing:
- net /Core/PB7: track 0.00 -> 38.9 mm, vias 0 -> 1
- net /Core/PB5: track 0.00 -> 36.0 mm, vias 0 -> 1
- net /Core/SWCLK: track 0.00 -> 35.4 mm, vias 0 -> 2
- net /Core/SWDIO: track 0.00 -> 34.6 mm, vias 0 -> 2
- net /Core/PB6: track 0.00 -> 34.5 mm, vias 0 -> 1
- net /Core/NRST: track 0.00 -> 34.1 mm, vias 0 -> 1
- net VSS: track 0.00 -> 33.6 mm
- net /Core/UART3_TX: track 0.00 -> 32.4 mm
- net /Core/PB3: track 0.00 -> 31.7 mm, vias 0 -> 1
- net /Core/PB4: track 0.00 -> 30.9 mm, vias 0 -> 1
- net /Core/UART3_RX: track 0.00 -> 30.4 mm
- net /Core/PA15: track 0.00 -> 28.8 mm, vias 0 -> 1
- net /Core/PA0: track 0.00 -> 26.7 mm
- net +5V: track 0.00 -> 26.4 mm
- net /Core/PA8: track 0.00 -> 22.1 mm, vias 0 -> 1
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
Commit message: PCB基本完成
Parts:
- C1, C12, C15, C8: footprint Library:C_0603_1608Metric_Pad1.08x0.95mm_HandSolder -> Capacitor_SMD:C_0603_1608Metric_Pad1.08x0.95mm_HandSolder
- C10, C11, C13, C14, C16, C2, C3, C4, C5, C6, C7, C9: footprint Library:C_0402_1005Metric_Pad0.74x0.62mm_HandSolder -> Capacitor_SMD:C_0402_1005Metric_Pad0.74x0.62mm_HandSolder
- C17: footprint Library:C_1210_3225Metric_Pad1.33x2.70mm_HandSolder -> Capacitor_SMD:C_1210_3225Metric_Pad1.33x2.70mm_HandSolder
- D1, D2, D3, D4, D5: footprint Library:LED_0805_2012Metric_Pad1.15x1.40mm_HandSolder -> LED_SMD:LED_0805_2012Metric_Pad1.15x1.40mm_HandSolder
- IC1: footprint Library:LQFP-32_7x7mm_P0.8mm -> Package_QFP:LQFP-32_7x7mm_P0.8mm
- J1, J3: footprint Library:PinHeader_1x04_P2.54mm_Vertical -> Connector_PinHeader_2.54mm:PinHeader_1x04_P2.54mm_Vertical
- J2: footprint Library:PinHeader_2x10_P2.54mm_Vertical -> Connector_PinHeader_2.54mm:PinHeader_2x10_P2.54mm_Vertical
- J5: footprint Library:JST_NV_B02P-NV_1x02_P5.00mm_Vertical -> Connector_JST:JST_NV_B02P-NV_1x02_P5.00mm_Vertical
- R1, R10, R15, R17, R2, R3, R4, R5, R6, R7, R8, R9: footprint Library:R_0402_1005Metric_Pad0.72x0.64mm_HandSolder -> Resistor_SMD:R_0402_1005Metric_Pad0.72x0.64mm_HandSolder
- R11, R12, R13: footprint Library:R_0805_2012Metric_Pad1.20x1.40mm_HandSolder -> Resistor_SMD:R_0805_2012Metric_Pad1.20x1.40mm_HandSolder
- R14, R16: footprint Library:R_1210_3225Metric_Pad1.30x2.65mm_HandSolder -> Resistor_SMD:R_1210_3225Metric_Pad1.30x2.65mm_HandSolder
- SW1, SW2: footprint Library:SW_PUSH_6mm_H5mm -> Button_Switch_THT:SW_PUSH_6mm_H5mm
- U1: footprint Library:SOIC-16_3.9x9.9mm_P1.27mm -> Package_SO:SOIC-16_3.9x9.9mm_P1.27mm
- U2: footprint Library:SOT-223-3_TabPin2 -> Package_TO_SOT_SMD:SOT-223-3_TabPin2
- U3: footprint Library:SOIC-8_3.9x4.9mm_P1.27mm -> Package_SO:SOIC-8_3.9x4.9mm_P1.27mm
- Y1: footprint Library:Crystal_HC49-U_Vertical -> Crystal:Crystal_HC49-U_Vertical
- moved R12 57.4 mm to (168.0, 115.1)
- moved U2 52.2 mm to (161.4, 116.1), turned to 0 degrees
- moved C14 46.9 mm to (155.7, 115.5), turned to 90 degrees
- moved C15 44.5 mm to (154.2, 115.2), turned to 90 degrees
- moved C13 42.3 mm to (155.6, 118.9), turned to -90 degrees
- moved C12 41.0 mm to (154.2, 119.2), turned to -90 degrees
- moved R13 35.3 mm to (149.4, 118.7), turned to 180 degrees
- moved C17 9.58 mm to (168.6, 119.9)
- moved R11 9.46 mm to (170.3, 115.1), turned to 90 degrees
- moved C1 7.11 mm to (148.7, 114.7), turned to -90 degrees
- moved R16 6.27 mm to (168.6, 129.4)
- moved C16 6.27 mm to (156.2, 126.4)
- moved R14 6.27 mm to (168.6, 123.3)
- moved R15 6.27 mm to (159.5, 123.1)
- moved R17 6.27 mm to (162.1, 123.1)
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Connections:
- J1 pad 1: VCC -> +5V
- J1 pad 4: VSS -> GND
Routing:
- net +5V: track 26.4 -> 120.1 mm, vias 0 -> 3
- net VDD: track 9.47 -> 65.1 mm, vias 0 -> 5
- net VCC: track 0.00 -> 46.5 mm, vias 0 -> 1
- net VSS: track 33.6 -> 77.8 mm, vias 0 -> 8
- net /CAN/CAN_TX: track 17.2 -> 27.2 mm
- net Net-(J4-CC2): track 0.00 -> 8.44 mm, vias 0 -> 2
- net /CAN/CAN_RX: track 20.7 -> 28.6 mm
- net GND: track 13.2 -> 17.4 mm
- net /Core/PA15: track 28.8 -> 30.9 mm
- net /Core/BOOT0: track 8.99 -> 7.66 mm
Other:
- board outline added: 59.6 x 43.6 mm

Commit message: PCB初稿与Gerber
Parts:
- moved C11 0.20 mm to (171.3, 100.6)
- moved R10 0.20 mm to (171.4, 98.4)
- moved R9 0.20 mm to (171.4, 99.4)
Routing:
- net GND: track 17.4 -> 51.4 mm, vias 0 -> 11
- net /Core/PA8: track 22.6 -> 25.2 mm
- net VDD: track 65.1 -> 67.5 mm
- net /Core/NRST: track 34.1 -> 32.7 mm
- net VSS: track 77.8 -> 78.8 mm, vias 8 -> 9
- net Net-(J5-Pin_2): track 15.9 -> 15.1 mm
- net Net-(J5-Pin_1): track 16.1 -> 15.3 mm
- net +5V: track 120.1 -> 119.4 mm, vias 3 -> 2
- net Net-(D4-K): track 22.1 -> 21.6 mm
- net Net-(D2-K): track 4.56 -> 4.00 mm
- net Net-(D1-K): track 4.60 -> 4.04 mm
- net /USB/D-: vias 1 -> 0
- added copper zone on B.Cu, net GND
- added copper zone on B.Cu, net VSS
Other:
- outline, holes or cut-outs redrawn
